File: HARDWARE/Projeto_Temperatura.brd (EAGLE design)
At the start: 60.3 x 36.5 mm, 14 parts, among them J1 DCJ0202, U1 328P

Commit message: commit
Parts:
- removed J1: DCJ0202, con-jack:DCJ0202
- added CON1: (no value), con-jack:DCJ0202
- added REG1: REGULADOR, ReguladoresTensao:REGULADOR
- BZ1: value F/CM12P -> (none)
- moved R3 0.63 mm to (39.4, 15.6)
- renumbered S1 to SWITCH, SG1 to BZ1, U$1 to SENSOR1, U1 to MICRO1
Connections:
- removed net N$4: DISPLAY_I2C.1, J1.1, MICRO1.7, R1.2, R3.1, R5.2, SENSOR1.VDD
- new net N$12: DISPLAY_I2C.1, MICRO1.7, R1.2, R3.1, R5.2, REG1.7, REG1.8, SENSOR1.VDD
- new net N$14: CON1.1, REG1.3, REG1.4
- new net N$15: CON1.2, CON1.3, REG1.1, REG1.2
- net GND: now also REG1.5, REG1.6; no longer J1.2, J1.3
Routing:
- net N$12: track 0.00 -> 191.1 mm
- net N$4: track 181.5 -> 0.00 mm
- net N$15: track 0.00 -> 29.5 mm
- net GND: track 175.6 -> 202.5 mm
- net N$14: track 0.00 -> 12.8 mm
- net N$2: track 51.5 -> 62.0 mm
- net N$6: track 35.3 -> 33.3 mm
- added copper zone on layer 16, net GND
Other:
- board size 60.3 x 36.5 mm -> 77.1 x 36.5 mm
- board text added: "BZ1"
- board text added: "REG1"
