File: HARDWARE/Projeto_Temperatura.sch (EAGLE design)
At the start: 14 parts, among them J1 DCJ0202, U1 328P

Commit message: commit
Parts:
- removed J1: DCJ0202, con-jack:DCJ0202
- removed S1: MOMENTARY-SWITCH-SPST-PTH-RIGHT-ANGLE-KIT, SparkFun-Switches:MOMENTARY-SWITCH-SPST-PTH-RIGHT-ANGLE-KIT
- removed SG1: F/CM12P, buzzer:F/CM12P
- removed U$1: DS18B20, Projeto1:DS18B20
- removed U1: 328P, SparkFun-IC-Microcontroller:ATMEGA328P_PDIP
- added BZ1: F/CM12P, buzzer:F/CM12P
- added CON1: DCJ0202, con-jack:DCJ0202
- added MICRO1: 328P, SparkFun-IC-Microcontroller:ATMEGA328P_PDIP
- added REG1: REGULADOR, ReguladoresTensao:REGULADOR
- added SENSOR1: DS18B20, Projeto1:DS18B20
- added SWITCH: MOMENTARY-SWITCH-SPST-PTH-RIGHT-ANGLE-KIT, SparkFun-Switches:MOMENTARY-SWITCH-SPST-PTH-RIGHT-ANGLE-KIT
Connections:
- removed net N$4: DISPLAY_I2C.1, J1.1, R1.2, R3.1, R5.2, U$1.3, U1.VCC
- new net N$12: DISPLAY_I2C.1, MICRO1.VCC, R1.2, R3.1, R5.2, REG1.OUT+, REG1.OUT+., SENSOR1.3
- new net N$14: CON1.1, REG1.IN+, REG1.IN+.
- new net N$15: CON1.2, CON1.3, REG1.IN-, REG1.IN-.
- net GND: now also BZ1.2, MICRO1.GND@1, REG1.OUT-, REG1.OUT-., SENSOR1.1, SWITCH.1; no longer J1.2, J1.3, S1.1, SG1.2, U$1.1, U1.GND@1
- net N$10: now also MICRO1.PC4(ADC4/SDA); no longer U1.PC4(ADC4/SDA)
- net N$11: now also MICRO1.PC5(ADC5/SCL); no longer U1.PC5(ADC5/SCL)
- net N$2: now also MICRO1.PD7(AIN1); no longer U1.PD7(AIN1)
- net N$6: now also MICRO1.PC3(ADC3), SENSOR1.2; no longer U$1.2, U1.PC3(ADC3)
- net N$7: now also MICRO1.PB3(MOSI/OC2); no longer U1.PB3(MOSI/OC2)
- net N$8: now also BZ1.1, MICRO1.PD2(INT0); no longer SG1.1, U1.PD2(INT0)
- net N$9: now also MICRO1.PB2(SS/OC1B), SWITCH.2; no longer S1.2, U1.PB2(SS/OC1B)
Other:
- note added: "REG1"
- moved on the sheet: DISPLAY_I2C, LED1, LED2, LED3, R1, R2, R3, R4, R5
